File: Hardware/Circuit/MiniVerb.kicad_pcb (KiCad board)
At the start: 2 copper layers, 40 x 97.5 mm, 50 parts, among them J1 IDC_2x05, U1 TL074, U2 TL074

Commit message: initial panel
Parts:
- added REF**: PanelHole_AudioJack_3.5mm, benjiaomodular:PanelHole_AudioJack_3.5mm, F.Cu at (155.0, 135.5)
- added REF**: PanelHole_Potentiometer_RV09, benjiaomodular:PanelHole_Potentiometer_RV09, F.Cu at (147.4, 103.6)
- added REF**: PanelHole_Potentiometer_RV09, benjiaomodular:PanelHole_Potentiometer_RV09, F.Cu at (127.7, 83.6)
- added REF**: PanelHole_AudioJack_3.5mm, benjiaomodular:PanelHole_AudioJack_3.5mm, F.Cu at (125.0, 135.5)
- added REF**: PanelHole_Potentiometer_RV09, benjiaomodular:PanelHole_Potentiometer_RV09, F.Cu at (127.7, 103.5)
- added REF**: PanelHole_Potentiometer_RV09, benjiaomodular:PanelHole_Potentiometer_RV09, F.Cu at (147.4, 63.5)
- added REF**: PanelHole_Potentiometer_RV09, benjiaomodular:PanelHole_Potentiometer_RV09, F.Cu at (127.7, 63.5)
- added REF**: PanelHole_AudioJack_3.5mm, benjiaomodular:PanelHole_AudioJack_3.5mm, F.Cu at (145.0, 135.5)
- added REF**: PanelHole_AudioJack_3.5mm, benjiaomodular:PanelHole_AudioJack_3.5mm, F.Cu at (135.0, 135.5)
- moved AUDIO_IN1 1.00 mm to (79.9, 135.4)
- moved AUDIO_IN2 1.00 mm to (90.0, 135.4)
- moved AUDIO_OUT1 1.00 mm to (100.0, 135.4)
- moved AUDIO_OUT2 1.00 mm to (110.0, 135.4)
- moved D1 0.11 mm to (103.8, 113.9)
- moved REF** 0.08 mm to (120.0, 32.0)
- moved POT_FBK1 0.08 mm to (82.7, 83.6)
Routing:
- net WET: track 15.4 -> 24.3 mm
- net 3V3_A: track 134.3 -> 137.0 mm
- net LPF: track 44.7 -> 46.3 mm
- net INT_AUDIO_OUT1: track 20.4 -> 19.4 mm
- net GND: vias 0 -> 237
- net (no net): vias 0 -> 1
- added copper zone on F.Cu, net (none)
Other:
- board size 40 x 97.5 mm -> 85 x 128.5 mm
