File: Hardware/MiniVerb v2/Circuit/MiniVerb.kicad_sch (KiCad schematic)
At the start: 44 parts, among them J1 IDC_2x05, U1 TL074, U2 LM4040LP-10, U3 MCP6001-OT

Commit message: Added BOM
Parts:
- C1, C2, C4: Manufacturers Name (none) -> YAGEO; Manufacturers Part Number (none) -> CC0603JRNPO9BN470; Mfg # (none) -> CC0603JRNPO9BN470
- C13, C7, C8, C9: Manufacturers Name (none) -> YAGEO; Manufacturers Part Number (none) -> CC0805KRX7R9BB104; Mfg # (none) -> CC0805KRX7R9BB104
- C14: Manufacturers Name (none) -> YAGEO; Manufacturers Part Number (none) -> CC0603JRX7R9BB103; Mfg # (none) -> CC0603JRX7R9BB103
- J1: Package Straight,P=2.54mm -> (none)
- R1, R7: Manufacturers Name (none) -> YAGEO; Manufacturers Part Number (none) -> AC0603FR-0710KL; Mfg # (none) -> AC0603FR-0710KL
- R10, R9: Manufacturers Name (none) -> YAGEO; Manufacturers Part Number (none) -> RC0603FR-071KL; Mfg # (none) -> RC0603FR-071KL
- R11: Package 0603 -> (none)
- R16, R2, R3, R4, R5, R6, R8: Manufacturers Name (none) -> YAGEO; Manufacturers Part Number (none) -> RC0603FR-07100KL; Mfg # (none) -> RC0603FR-07100KL
- U2: Manufacturers Name (none) -> Texas Instruments; Manufacturers Part Number (none) -> LM4040CIM3-10.0/NOPB; Mfg # (none) -> LM4040CIM3-10.0/NOPB
- U3: Manufacturers Name (none) -> Microchip Technology / Atmel; Manufacturers Part Number (none) -> MCP6001UT-I/OT; Mfg # (none) -> MCP6001UT-I/OT
