File: Hardware/MiniVerb v1.1/Circuit/power.kicad_sch (KiCad schematic)
At the start: 11 parts, among them J1 IDC_2x05, U1 TL074, U2 TL074

Commit message: Updated BOM
Parts:
- C10, C9: Manufacturers Name (none) -> KEMET; Manufacturers Part Number (none) -> ESH107M010AC3AA
- C11, C12, C13, C14: Manufacturers Name (none) -> KEMET; Manufacturers Part Number (none) -> MMK5104K50J01L4BULK
- R21: Manufacturers Name YAGEO -> KOA Speer; Manufacturers Part Number AC0603FR-0710KL -> MF1/4DC1002F; Package 0603 -> (none); Part Description Thick Film Resistors - SMD 10 kOhms 100mW 0603 1% AEC-Q200 -> (none)
- U1, U2: Manufacturers Name (none) -> Texas Instruments; Manufacturers Part Number (none) -> TL074BCN
Changed lines of the file:
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@@
+      (effects (font (size 1.27 1.27)) hide)
+    )
+    (property "Manufacturers Name" "KEMET" (id 4) (at 182.118 83.566 0)
+      (effects (font (size 1.27 1.27)) hide)
+    )
+    (property "Manufacturers Part Number" "MMK5104K50J01L4BULK" (id 5) (at 182.118 83.566 0)
       (effects (font (size 1.27 1.27)) hide)
     )
@@
       (effects (font (size 1.27 1.27)) hide)
     )
-    (property "Manufacturers Part Number" "AC0603FR-0710KL" (id 6) (at 188.722 69.977 0)
-      (effects (font (size 1.27 1.27)) hide)
-    )
-    (property "Manufacturers Name" "YAGEO" (id 7) (at 188.722 69.977 0)
-      (effects (font (size 1.27 1.27)) hide)
-    )
-    (property "Package" "0603" (id 8) (at 188.722 69.977 0)
+    (property "Manufacturers Part Number" "MF1/4DC1002F" (id 6) (at 188.722 69.977 0)
+      (effects (font (size 1.27 1.27)) hide)
+    )
+    (property "Manufacturers Name" "KOA Speer" (id 7) (at 188.722 69.977 0)
+      (effects (font (size 1.27 1.27)) hide)
+    )
+    (property "Package" "" (id 8) (at 188.722 69.977 0)
       (effects (font (size 1.27 1.27)) hide)
     )
@@
       (effects (font (size 1.27 1.27)) hide)
     )
-    (property "Part Description" "Thick Film Resistors - SMD 10 kOhms 100mW 0603 1% AEC-Q200 " (id 10) (at 188.722 69.977 0)
+    (property "Part Description" "" (id 10) (at 188.722 69.977 0)
       (effects (font (size 1.27 1.27)) hide)
     )
@@
       (effects (font (size 1.27 1.27)) hide)
     )
+    (property "Manufacturers Name" "KEMET" (id 4) (at 170.18 74.422 0)
+      (effects (font (size 1.27 1.27)) hide)
+    )
+    (property "Manufacturers Part Number" "MMK5104K50J01L4BULK" (id 5) (at 170.18 74.422 0)
+      (effects (font (size 1.27 1.27)) hide)
+    )
     (pin "1")
     (pin "2")
@@
     )
     (property "Datasheet" "http://www.ti.com/lit/ds/symlink/tl071.pdf" (id 3) (at 149.352 73.152 0)
+      (effects (font (size 1.27 1.27)) hide)
+    )
+    (property "Manufacturers Name" "Texas Instruments" (id 4) (at 148.082 78.232 0)
+      (effects (font (size 1.27 1.27)) hide)
+    )
+    (property "Manufacturers Part Number" "TL074BCN" (id 5) (at 148.082 78.232 0)
       (effects (font (size 1.27 1.27)) hide)
     )
@@
       (effects (font (size 1.27 1.27)) hide)
     )
+    (property "Manufacturers Name" "KEMET" (id 4) (at 157.607 83.185 0)
+      (effects (font (size 1.27 1.27)) hide)
+    )
+    (property "Manufacturers Part Number" "ESH107M010AC3AA" (id 5) (at 157.607 83.185 0)
+      (effects (font (size 1.27 1.27)) hide)
+    )
     (pin "1")
     (pin "2")
@@
       (effects (font (size 1.27 1.27)) hide)
     )
+    (property "Manufacturers Name" "KEMET" (id 4) (at 170.18 83.312 0)
+      (effects (font (size 1.27 1.27)) hide)
+    )
+    (property "Manufacturers Part Number" "MMK5104K50J01L4BULK" (id 5) (at 170.18 83.312 0)
+      (effects (font (size 1.27 1.27)) hide)
+    )
     (pin "1")
     (pin "2")
@@
     )
     (property "Datasheet" "http://www.ti.com/lit/ds/symlink/tl071.pdf" (id 3) (at 136.017 73.152 0)
+      (effects (font (size 1.27 1.27)) hide)
+    )
+    (property "Manufacturers Name" "Texas Instruments" (id 4) (at 134.747 78.232 0)
+      (effects (font (size 1.27 1.27)) hide)
+    )
+    (property "Manufacturers Part Number" "TL074BCN" (id 5) (at 134.747 78.232 0)
       (effects (font (size 1.27 1.27)) hide)
     )
@@
       (effects (font (size 1.27 1.27)) hide)
     )
+    (property "Manufacturers Name" "KEMET" (id 4) (at 182.118 74.168 0)
+      (effects (font (size 1.27 1.27)) hide)
+    )
+    (property "Manufacturers Part Number" "MMK5104K50J01L4BULK" (id 5) (at 182.118 74.168 0)
+      (effects (font (size 1.27 1.27)) hide)
+    )
     (pin "1")
     (pin "2")
@@
       (effects (font (size 1.27 1.27)) hide)
     )
+    (property "Manufacturers Name" "KEMET" (id 4) (at 157.607 74.422 0)
+      (effects (font (size 1.27 1.27)) hide)
+    )
+    (property "Manufacturers Part Number" "ESH107M010AC3AA" (id 5) (at 157.607 74.422 0)
+      (effects (font (size 1.27 1.27)) hide)
+    )
