File: Hardware/MiniVerb v2.0/Circuit/MiniVerb.kicad_pcb (KiCad board)
At the start: 2 copper layers, 47.9 x 128.5 mm, 51 parts, among them J1 IDC_2x05, U1 TL074, U2 LM4040LP-10, U3 MCP6001-OT

Commit message: Updated BOM
Parts:
- C3: value 580pF -> 680pF
