File: Hardware/MiniVerb v2.0/Circuit/MiniVerb.kicad_sch (KiCad schematic)
At the start: 44 parts, among them J1 IDC_2x05, U1 TL074, U2 LM4040LP-10, U3 MCP6001-OT

Commit message: Updated BOM
Parts:
- A1: Manufacturers Name (none) -> Electro-Smith
- AUDIO_IN1, AUDIO_OUT1, CV1_IN1: Manufacturers Name (none) -> Tayda Electronics; Manufacturers Part Number (none) -> PJ-3001F
- C3: value 580pF -> 680pF; Manufacturers Name (none) -> Vishay / Vitramon; Manufacturers Part Number (none) -> VJ0603Y681KXAAC
- C5, C6: Manufacturers Name (none) -> Murata Electronics; Manufacturers Part Number (none) -> GRM219R60J476ME44D
- FEEDBACK_POT1, LEVEL_POT1, MOD_POT1: Manufacturers Name (none) -> Alpha (Taiwan); Manufacturers Part Number (none) -> RD901F-40-15R1-B10K; Part Description (none) -> 10K OHM Linear Taper Potentiometer Round Shaft PCB 9mm
- R12: Manufacturers Name (none) -> TE Connectivity / Holsworthy; Manufacturers Part Number (none) -> CRG0603F330R
- R14: Manufacturers Name (none) -> Bourns; Manufacturers Part Number (none) -> CR0603-FX-2003ELF
- R17: Manufacturers Name (none) -> YAGEO; Manufacturers Part Number (none) -> RC0603FR-0766K5L
- U1: Manufacturers Name (none) -> Texas Instruments; Manufacturers Part Number (none) -> TL074HIDYYR
Other:
- note added: "Audio Inputs"
- note added: "CV Input"
- note removed: "Input"
- moved on the sheet: C13, C14, C5, C6, C7, C8, C9, CV1_IN1, D1, J1, R11, R12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
