File: Hardware/MiniVerb v2.1/Circuit/MiniVerb.kicad_sch (KiCad schematic)
At the start: 47 parts, among them J1 IDC_2x05, U1 TL074, U2 LM4040DBZ-10, U3 MCP6001-OT

Commit message: cleanup and ibom
Parts:
- removed TP1: TP_12V, TestPoint:TestPoint_THTPad_1.0x1.0mm_Drill0.5mm, symbol Connector:TestPoint_Flag
- removed TP2: TP_-12V, TestPoint:TestPoint_THTPad_1.0x1.0mm_Drill0.5mm, symbol Connector:TestPoint_Flag
- removed TP3: TP_GND, TestPoint:TestPoint_Loop_D1.80mm_Drill1.0mm_Beaded, symbol Connector:TestPoint_Flag
- removed TP4: TP_-10V, TestPoint:TestPoint_THTPad_1.0x1.0mm_Drill0.5mm, symbol Connector:TestPoint_Flag
- removed TP5: TP_3.3V, TestPoint:TestPoint_THTPad_1.0x1.0mm_Drill0.5mm, symbol Connector:TestPoint_Flag
- removed TP7: TP_INPUT_BUFFER, TestPoint:TestPoint_THTPad_1.0x1.0mm_Drill0.5mm, symbol Connector:TestPoint_Flag
- FB1, FB2: renamed from FB?; footprint (none) -> Capacitor_SMD:C_0603_1608Metric_Pad1.08x0.95mm_HandSolder; Manufacturers Name (none) -> Wurth Elektronik; Manufacturers Part Number (none) -> 742792664
- FEEDBACK_POT1, LEVEL_POT1, MOD_POT1: footprint benjiaomodular:Potentiometer_RV09 -> benjiaomodular:Potentiometer_RV09_NoBracket
- R11: value 10k -> 220
- U2: Manufacturers Name (none) -> Texas Instruments; Manufacturers Part Number (none) -> LM4040CIM3-10.0/NOPB
- U3: Manufacturers Name (none) -> Microchip Technology / Atmel; Manufacturers Part Number (none) -> MCP6001T-E/OT
- gave numbers to parts that had none: 1
Connections:
- net +12V: no longer R11.2
- net LED: now reaches A1.30 (DAC1_OUT1)
- net LED: now also R11.2
- no-connect marks 33 -> 32
